File: v3-tx-shield-v3.4.kicad_pcb (KiCad board)
At the start: 2 copper layers, 116.8 x 58.4 mm, 109 parts, among them J1 Conn_01x08_Male, J2 Conn_01x02_Male, J3 Conn_01x02_Male, P1 Power, P2 Analog, P3 Digital, P4 Digital

Commit message: Final version
Parts:
- bjt-1, bjt-10, bjt-11, bjt-12, bjt-13, bjt-14, bjt-15, bjt-16, bjt-17, bjt-18, bjt-19, bjt-2, bjt-20, bjt-3, bjt-4, bjt-5, bjt-6, bjt-7, bjt-8, bjt-9: value MCH4020-RF -> BUT11A
- moved R-base-2 0.51 mm to (145.5, 104.6)
- moved R-base-3 0.44 mm to (155.7, 104.6)
- moved R-base-4 0.32 mm to (165.9, 104.6)
- moved R-base-1 0.19 mm to (135.4, 104.6)
Connections:
- bjt-1 pad 1: Net-(bjt-1-Pad1) -> Net-(R-base-1-Pad1)
- bjt-1 pad 2: GND -> Net-(bjt-1-Pad2)
- bjt-1 pad 3: Net-(R-base-1-Pad1) -> GND
- bjt-1 pad 4: GND -> (no net)
- bjt-10 pad 1: Net-(bjt-10-Pad1) -> Net-(R-base-10-Pad1)
- bjt-10 pad 2: GND -> Net-(bjt-10-Pad2)
- bjt-10 pad 3: Net-(R-base-10-Pad1) -> GND
- bjt-10 pad 4: GND -> (no net)
- bjt-11 pad 1: Net-(bjt-11-Pad1) -> Net-(R-base-11-Pad1)
- bjt-11 pad 2: GND -> Net-(bjt-11-Pad2)
- bjt-11 pad 3: Net-(R-base-11-Pad1) -> GND
- bjt-11 pad 4: GND -> (no net)
- bjt-12 pad 1: Net-(bjt-12-Pad1) -> Net-(R-base-12-Pad1)
- bjt-12 pad 2: GND -> Net-(bjt-12-Pad2)
- bjt-12 pad 3: Net-(R-base-12-Pad1) -> GND
- bjt-12 pad 4: GND -> (no net)
- bjt-13 pad 1: Net-(bjt-13-Pad1) -> Net-(R-base-13-Pad1)
- bjt-13 pad 2: GND -> Net-(bjt-13-Pad2)
- bjt-13 pad 3: Net-(R-base-13-Pad1) -> GND
- bjt-13 pad 4: GND -> (no net)
- bjt-14 pad 1: Net-(bjt-14-Pad1) -> Net-(R-base-14-Pad1)
- bjt-14 pad 2: GND -> Net-(bjt-14-Pad2)
- bjt-14 pad 3: Net-(R-base-14-Pad1) -> GND
- bjt-14 pad 4: GND -> (no net)
- bjt-15 pad 1: Net-(bjt-15-Pad1) -> Net-(R-base-15-Pad1)
- bjt-15 pad 2: GND -> Net-(bjt-15-Pad2)
- bjt-15 pad 3: Net-(R-base-15-Pad1) -> GND
- bjt-15 pad 4: GND -> (no net)
- bjt-16 pad 1: Net-(bjt-16-Pad1) -> Net-(R-base-16-Pad1)
- bjt-16 pad 2: GND -> Net-(bjt-16-Pad2)
- bjt-16 pad 3: Net-(R-base-16-Pad1) -> GND
- bjt-16 pad 4: GND -> (no net)
- bjt-17 pad 1: Net-(bjt-17-Pad1) -> Net-(R-base-17-Pad1)
- bjt-17 pad 2: GND -> Net-(bjt-17-Pad2)
- bjt-17 pad 3: Net-(R-base-17-Pad1) -> GND
- bjt-17 pad 4: GND -> (no net)
- bjt-18 pad 1: Net-(bjt-18-Pad1) -> Net-(R-base-18-Pad1)
- bjt-18 pad 2: GND -> Net-(bjt-18-Pad2)
- bjt-18 pad 3: Net-(R-base-18-Pad1) -> GND
- bjt-18 pad 4: GND -> (no net)
- bjt-19 pad 1: Net-(bjt-19-Pad1) -> Net-(R-base-19-Pad1)
- bjt-19 pad 2: GND -> Net-(bjt-19-Pad2)
- bjt-19 pad 3: Net-(R-base-19-Pad1) -> GND
- bjt-19 pad 4: GND -> (no net)
- bjt-2 pad 1: Net-(bjt-2-Pad1) -> Net-(R-base-2-Pad1)
- bjt-2 pad 2: GND -> Net-(bjt-2-Pad2)
- bjt-2 pad 3: Net-(R-base-2-Pad1) -> GND
- bjt-2 pad 4: GND -> (no net)
- bjt-20 pad 1: Net-(bjt-20-Pad1) -> Net-(R-base-20-Pad1)
- bjt-20 pad 2: GND -> Net-(bjt-20-Pad2)
- bjt-20 pad 3: Net-(R-base-20-Pad1) -> GND
- bjt-20 pad 4: GND -> (no net)
- bjt-3 pad 1: Net-(bjt-3-Pad1) -> Net-(R-base-3-Pad1)
- bjt-3 pad 2: GND -> Net-(bjt-3-Pad2)
- bjt-3 pad 3: Net-(R-base-3-Pad1) -> GND
- bjt-3 pad 4: GND -> (no net)
- bjt-4 pad 1: Net-(bjt-4-Pad1) -> Net-(R-base-4-Pad1)
- bjt-4 pad 2: GND -> Net-(bjt-4-Pad2)
- bjt-4 pad 3: Net-(R-base-4-Pad1) -> GND
- bjt-4 pad 4: GND -> (no net)
- bjt-5 pad 1: Net-(bjt-5-Pad1) -> Net-(R-base-5-Pad1)
- bjt-5 pad 2: GND -> Net-(bjt-5-Pad2)
- bjt-5 pad 3: Net-(R-base-5-Pad1) -> GND
- bjt-5 pad 4: GND -> (no net)
- bjt-6 pad 1: Net-(bjt-6-Pad1) -> Net-(R-base-6-Pad1)
- bjt-6 pad 2: GND -> Net-(bjt-6-Pad2)
- bjt-6 pad 3: Net-(R-base-6-Pad1) -> GND
- bjt-6 pad 4: GND -> (no net)
- bjt-7 pad 1: Net-(bjt-7-Pad1) -> Net-(R-base-7-Pad1)
- bjt-7 pad 2: GND -> Net-(bjt-7-Pad2)
- bjt-7 pad 3: Net-(R-base-7-Pad1) -> GND
- bjt-7 pad 4: GND -> (no net)
- bjt-8 pad 1: Net-(bjt-8-Pad1) -> Net-(R-base-8-Pad1)
- bjt-8 pad 2: GND -> Net-(bjt-8-Pad2)
- bjt-8 pad 3: Net-(R-base-8-Pad1) -> GND
- bjt-8 pad 4: GND -> (no net)
- bjt-9 pad 1: Net-(bjt-9-Pad1) -> Net-(R-base-9-Pad1)
- bjt-9 pad 2: GND -> Net-(bjt-9-Pad2)
- bjt-9 pad 3: Net-(R-base-9-Pad1) -> GND
- bjt-9 pad 4: GND -> (no net)
- tx-1 pad 2: Net-(bjt-1-Pad1) -> Net-(bjt-1-Pad2)
- tx-10 pad 2: Net-(bjt-10-Pad1) -> Net-(bjt-10-Pad2)
- tx-11 pad 2: Net-(bjt-11-Pad1) -> Net-(bjt-11-Pad2)
- tx-12 pad 2: Net-(bjt-12-Pad1) -> Net-(bjt-12-Pad2)
- tx-13 pad 2: Net-(bjt-13-Pad1) -> Net-(bjt-13-Pad2)
- tx-14 pad 2: Net-(bjt-14-Pad1) -> Net-(bjt-14-Pad2)
- tx-15 pad 2: Net-(bjt-15-Pad1) -> Net-(bjt-15-Pad2)
- tx-16 pad 2: Net-(bjt-16-Pad1) -> Net-(bjt-16-Pad2)
- tx-17 pad 2: Net-(bjt-17-Pad1) -> Net-(bjt-17-Pad2)
- tx-18 pad 2: Net-(bjt-18-Pad1) -> Net-(bjt-18-Pad2)
- tx-19 pad 2: Net-(bjt-19-Pad1) -> Net-(bjt-19-Pad2)
- tx-2 pad 2: Net-(bjt-2-Pad1) -> Net-(bjt-2-Pad2)
- tx-20 pad 2: Net-(bjt-20-Pad1) -> Net-(bjt-20-Pad2)
- tx-3 pad 2: Net-(bjt-3-Pad1) -> Net-(bjt-3-Pad2)
- tx-4 pad 2: Net-(bjt-4-Pad1) -> Net-(bjt-4-Pad2)
- tx-5 pad 2: Net-(bjt-5-Pad1) -> Net-(bjt-5-Pad2)
- tx-6 pad 2: Net-(bjt-6-Pad1) -> Net-(bjt-6-Pad2)
- tx-7 pad 2: Net-(bjt-7-Pad1) -> Net-(bjt-7-Pad2)
- tx-8 pad 2: Net-(bjt-8-Pad1) -> Net-(bjt-8-Pad2)
- tx-9 pad 2: Net-(bjt-9-Pad1) -> Net-(bjt-9-Pad2)
Routing:
- net Net-(bjt-18-Pad1): track 6.38 -> 0.00 mm
- net Net-(bjt-17-Pad1): track 6.38 -> 0.00 mm
- net Net-(bjt-16-Pad1): track 6.38 -> 0.00 mm
- net Net-(bjt-8-Pad1): track 6.38 -> 0.00 mm
- net Net-(bjt-7-Pad1): track 6.38 -> 0.00 mm
- net Net-(bjt-6-Pad1): track 6.38 -> 0.00 mm
- net Net-(bjt-20-Pad1): track 6.38 -> 0.00 mm
- net Net-(bjt-19-Pad1): track 6.38 -> 0.00 mm
- net Net-(bjt-15-Pad1): track 6.38 -> 0.00 mm
- net Net-(bjt-14-Pad1): track 6.38 -> 0.00 mm
- net Net-(bjt-13-Pad1): track 6.38 -> 0.00 mm
- net Net-(bjt-12-Pad1): track 6.38 -> 0.00 mm
- net Net-(bjt-11-Pad1): track 6.38 -> 0.00 mm
- net Net-(bjt-9-Pad1): track 6.38 -> 0.00 mm
- net Net-(bjt-5-Pad1): track 6.38 -> 0.00 mm
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